File: Split Keyboard.kicad_pcb (KiCad board)
At the start: 2 copper layers, 254 x 101.2 mm, 103 parts, among them SW1 SW_Push, SW10 SW_Push, SW11 SW_Push, SW12 SW_Push, SW13 SW_Push, SW14 SW_Push, SW15 SW_Push, SW16 SW_Push, SW17 SW_Push, SW18 SW_Push, SW19 SW_Push, SW2 SW_Push, SW20 SW_Push, SW21 SW_Push, SW22 SW_Push, SW23 SW_Push, SW24 SW_Push, SW25 SW_Push, SW26 SW_Push, SW27 SW_Push, SW28 SW_Push, SW29 SW_Push, SW3 SW_Push, SW30 SW_Push, SW31 SW_Push, SW32 SW_Push, SW33 SW_Push, SW34 SW_Push, SW35 SW_Push, SW36 SW_Push, SW37 SW_Push, SW38 SW_Push, SW39 SW_Push, SW4 SW_Push, SW40 SW_Push, SW41 SW_Push, SW42 SW_Push, SW5 SW_Push, SW6 SW_Push, SW7 SW_Push, SW8 SW_Push, SW9 SW_Push, U1 XIAO-nRF52840-SMD, U2 XIAO-nRF52840-SMD

Commit message: Configure Infinix split keyboard and update files
Parts:
- removed H3, H4: MountingHole, MountingHole:MountingHole_3.2mm_M3
- added C43: 1 mF, Capacitor_SMD:CP_Elec_10x10, F.Cu at (170.4, 118.4)
- added C44: 1 mF, Capacitor_SMD:CP_Elec_10x10, F.Cu at (142.2, 117.7)
- added D43: SK6812MINI-E, kicad-keyboard-parts.pretty-master:MX_SK6812MINI-E, F.Cu at (122.8, 92.3)
- added D44: SK6812MINI-E, kicad-keyboard-parts.pretty-master:MX_SK6812MINI-E, F.Cu at (190.7, 92.2)
- added D45: SK6812MINI-E, kicad-keyboard-parts.pretty-master:MX_SK6812MINI-E, F.Cu at (103.8, 89.4)
- added D46: SK6812MINI-E, kicad-keyboard-parts.pretty-master:MX_SK6812MINI-E, F.Cu at (209.7, 89.3)
- added D47: SK6812MINI-E, kicad-keyboard-parts.pretty-master:MX_SK6812MINI-E, F.Cu at (84.7, 86.3)
- added D48: SK6812MINI-E, kicad-keyboard-parts.pretty-master:MX_SK6812MINI-E, F.Cu at (228.8, 86.2)
- added D49: SK6812MINI-E, kicad-keyboard-parts.pretty-master:MX_SK6812MINI-E, F.Cu at (65.6, 89.3)
- added D50: SK6812MINI-E, kicad-keyboard-parts.pretty-master:MX_SK6812MINI-E, F.Cu at (247.7, 89.3)
- added D51: SK6812MINI-E, kicad-keyboard-parts.pretty-master:MX_SK6812MINI-E, F.Cu at (46.7, 92.3)
- added D52: SK6812MINI-E, kicad-keyboard-parts.pretty-master:MX_SK6812MINI-E, F.Cu at (266.9, 92.3)
- added D53: SK6812MINI-E, kicad-keyboard-parts.pretty-master:MX_SK6812MINI-E, F.Cu at (46.8, 116.2)
- added D54: SK6812MINI-E, kicad-keyboard-parts.pretty-master:MX_SK6812MINI-E, F.Cu at (65.8, 113.3)
- added D55: SK6812MINI-E, kicad-keyboard-parts.pretty-master:MX_SK6812MINI-E, F.Cu at (84.7, 110.3)
- added D56: SK6812MINI-E, kicad-keyboard-parts.pretty-master:MX_SK6812MINI-E, F.Cu at (103.7, 113.4)
- added D57: SK6812MINI-E, kicad-keyboard-parts.pretty-master:MX_SK6812MINI-E, F.Cu at (122.7, 116.4)
- added D58: SK6812MINI-E, kicad-keyboard-parts.pretty-master:MX_SK6812MINI-E, F.Cu at (266.9, 116.3)
- added D59: SK6812MINI-E, kicad-keyboard-parts.pretty-master:MX_SK6812MINI-E, F.Cu at (247.9, 113.3)
- added D60: SK6812MINI-E, kicad-keyboard-parts.pretty-master:MX_SK6812MINI-E, F.Cu at (228.8, 110.3)
- added D61: SK6812MINI-E, kicad-keyboard-parts.pretty-master:MX_SK6812MINI-E, F.Cu at (209.8, 113.3)
- added D62: SK6812MINI-E, kicad-keyboard-parts.pretty-master:MX_SK6812MINI-E, F.Cu at (190.8, 116.3)
- added D63: SK6812MINI-E, kicad-keyboard-parts.pretty-master:MX_SK6812MINI-E, F.Cu at (122.8, 140.3)
- added D64: SK6812MINI-E, kicad-keyboard-parts.pretty-master:MX_SK6812MINI-E, F.Cu at (103.6, 137.4)
- added D65: SK6812MINI-E, kicad-keyboard-parts.pretty-master:MX_SK6812MINI-E, F.Cu at (84.7, 134.4)
- added D66: SK6812MINI-E, kicad-keyboard-parts.pretty-master:MX_SK6812MINI-E, F.Cu at (65.8, 137.5)
- added D67: SK6812MINI-E, kicad-keyboard-parts.pretty-master:MX_SK6812MINI-E, F.Cu at (46.9, 140.4)
- added D68: SK6812MINI-E, kicad-keyboard-parts.pretty-master:MX_SK6812MINI-E, F.Cu at (190.7, 140.4)
- added D69: SK6812MINI-E, kicad-keyboard-parts.pretty-master:MX_SK6812MINI-E, F.Cu at (209.7, 137.3)
- added D70: SK6812MINI-E, kicad-keyboard-parts.pretty-master:MX_SK6812MINI-E, F.Cu at (228.6, 134.3)
- added D71: SK6812MINI-E, kicad-keyboard-parts.pretty-master:MX_SK6812MINI-E, F.Cu at (247.7, 137.4)
- added D72: SK6812MINI-E, kicad-keyboard-parts.pretty-master:MX_SK6812MINI-E, F.Cu at (266.8, 140.4)
- added D73: SK6812MINI-E, kicad-keyboard-parts.pretty-master:MX_SK6812MINI-E, F.Cu at (46.6, 164.5)
- added D74: SK6812MINI-E, kicad-keyboard-parts.pretty-master:MX_SK6812MINI-E, F.Cu at (65.7, 161.5)
- added D75: SK6812MINI-E, kicad-keyboard-parts.pretty-master:MX_SK6812MINI-E, F.Cu at (84.7, 158.4)
- added D76: SK6812MINI-E, kicad-keyboard-parts.pretty-master:MX_SK6812MINI-E, F.Cu at (103.7, 161.4)
- added D77: SK6812MINI-E, kicad-keyboard-parts.pretty-master:MX_SK6812MINI-E, F.Cu at (122.7, 164.4)
- added D78: SK6812MINI-E, kicad-keyboard-parts.pretty-master:MX_SK6812MINI-E, F.Cu at (266.7, 164.4)
- added D79: SK6812MINI-E, kicad-keyboard-parts.pretty-master:MX_SK6812MINI-E, F.Cu at (247.8, 161.5)
- added D80: SK6812MINI-E, kicad-keyboard-parts.pretty-master:MX_SK6812MINI-E, F.Cu at (228.8, 158.4)
- added D81: SK6812MINI-E, kicad-keyboard-parts.pretty-master:MX_SK6812MINI-E, F.Cu at (209.7, 161.5)
- added D82: SK6812MINI-E, kicad-keyboard-parts.pretty-master:MX_SK6812MINI-E, F.Cu at (190.7, 164.3)
- added D83: SK6812MINI-E, kicad-keyboard-parts.pretty-master:MX_SK6812MINI-E, F.Cu at (141.8, 166.4)
- added D84: SK6812MINI-E, kicad-keyboard-parts.pretty-master:MX_SK6812MINI-E, F.Cu at (171.6, 166.3)
- added H5: MountingHole, MountingHole:MountingHole_3.2mm_M3, F.Cu at (161.7, 175.0)
- added H6: MountingHole, MountingHole:MountingHole_3.2mm_M3, F.Cu at (151.8, 174.9)
- added R5: 330, Resistor_SMD:R_1206_3216Metric, B.Cu at (127.2, 81.1)
- added R6: 330, Resistor_SMD:R_1206_3216Metric, B.Cu at (188.6, 81.1)
- R1, R2: footprint Resistor_SMD:R_0805_2012Metric -> Resistor_SMD:R_0603_1608Metric
- R3, R4: value 2m -> 2M
- SW1, SW10, SW11, SW12, SW13, SW14, SW15, SW16, SW17, SW18, SW19, SW2, SW20, SW21, SW22, SW23, SW24, SW25, SW26, SW27, SW28, SW29, SW3, SW30, SW31, SW32, SW33, SW34, SW35, SW36, SW37, SW38, SW39, SW4, SW40, SW41, SW42, SW5, SW6, SW7, SW8, SW9: footprint Button_Switch_Keyboard:SW_Cherry_MX_1.00u_PCB -> PCM_marbastlib-xp-mx:SW_Cherry_MX_1.00u_PCB
- TP1, TP2, TP3, TP4: moved to B.Cu
- U1, U2: footprint Seeed_Studio_XIAO_Series:XIAO-nRF52840-SMD -> New_XIAO_Series_Footprints:XIAO-nRF52840-SMD
- moved U1 51.9 mm to (136.2, 97.5)
- moved R4 40.9 mm to (168.1, 99.7), turned to -90 degrees
- moved R2 40.9 mm to (166.2, 99.7), turned to 90 degrees
- moved TP2 28.0 mm to (166.5, 107.0)
- moved TP4 27.9 mm to (170.4, 107.1), turned to 180 degrees
- moved R1 27.7 mm to (145.9, 99.2), turned to 90 degrees
- moved R3 26.3 mm to (144.0, 99.3), turned to -90 degrees
- moved D41 20.0 mm to (127.4, 175.4)
- moved U2 19.2 mm to (160.6, 97.5), turned to 0 degrees
- moved TP1 15.1 mm to (146.3, 106.9)
- moved TP3 11.1 mm to (142.5, 106.8)
- moved REF** 10.9 mm to (157.8, 164.6)
- moved D42 10.9 mm to (184.7, 175.4)
- moved D13 6.00 mm to (86.9, 121.8)
- moved D18 6.00 mm to (230.8, 121.8)
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Connections:
- U1 pad 12: unconnected-(U1-3V3_OUT-Pad12) -> +3.3V
- U1 pad 18: unconnected-(U1-GND-Pad18) -> GND
- U1 pad 21: unconnected-(U1-NFC1-Pad21) -> LED DATA
- U2 pad 12: unconnected-(U2-3V3_OUT-Pad12) -> +3.3V
- U2 pad 18: unconnected-(U2-GND-Pad18) -> GND
- U2 pad 21: unconnected-(U2-NFC1-Pad21) -> LED DATA
Routing:
- net GND: track 4.67 -> 277.2 mm, vias 7 -> 39
- net LED DATA: track 0.00 -> 52.4 mm, vias 0 -> 2
- net /left/ROW 3: track 128.7 -> 180.7 mm
- net /left/ROW 4: track 35.9 -> 83.7 mm, vias 2 -> 0
- net /left/ROW 2: track 112.2 -> 155.9 mm, vias 0 -> 6
- net /right/COL 3: track 143.4 -> 182.3 mm, vias 0 -> 1
- net +3.3V: track 0.00 -> 38.8 mm, vias 0 -> 16
- net /right/COL 0: track 83.2 -> 119.3 mm, vias 0 -> 1
- net /right/COL 2: track 124.5 -> 158.0 mm, vias 0 -> 1
- net /right/COL 1: track 106.4 -> 138.6 mm, vias 0 -> 1
- net Net-(D74-DOUT): track 0.00 -> 30.6 mm
- net Net-(D54-DOUT): track 0.00 -> 30.4 mm
- net Net-(D44-DOUT): track 0.00 -> 30.3 mm
- net Net-(D53-DOUT): track 0.00 -> 30.2 mm
- net Net-(D73-DOUT): track 0.00 -> 30.2 mm
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- added copper zone on B.Cu, net +3.3V
- removed copper zone on B.Cu, net GND
Other:
- board size 254 x 101.2 mm -> 255.2 x 104.3 mm
