File: side.kicad_sch (KiCad schematic)
At the start: 50 parts, among them SW1 SW_Push, SW11 SW_Push, SW12 SW_Push, SW13 SW_Push, SW14 SW_Push, SW15 SW_Push, SW21 SW_Push, SW22 SW_Push, SW23 SW_Push, SW24 SW_Push, SW25 SW_Push, SW3 SW_Push, SW31 SW_Push, SW32 SW_Push, SW33 SW_Push, SW34 SW_Push, SW35 SW_Push, SW41 SW_Push, SW5 SW_Push, SW6 SW_Push, SW9 SW_Push, U1 XIAO-nRF52840-SMD

Commit message: Add Infinix ZMK shield
Parts:
- R3: value 2m -> 2M
Changed lines of the file:
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@@
 			)
 		)
-		(property "Value" "2m"
+		(property "Value" "2M"
 			(at 185.42 130.81 90)
 			(show_name no)

Commit message: Configure Infinix split keyboard and update files
Parts:
- added C43: 1 mF, Capacitor_SMD:CP_Elec_10x10, symbol Device:C
- added D43, D45, D47, D49, D51, D53, D54, D55, D56, D57, D63, D64, D65, D66, D67, D73, D74, D75, D76, D77, D83: SK6812MINI-E, kicad-keyboard-parts.pretty-master:MX_SK6812MINI-E, symbol LED:SK6812MINI-E
- added R5: 330, Resistor_SMD:R_1206_3216Metric, symbol Device:R
- R1: footprint Resistor_SMD:R_0805_2012Metric -> Resistor_SMD:R_0603_1608Metric
- U1: footprint Seeed_Studio_XIAO_Series:XIAO-nRF52840-SMD -> New_XIAO_Series_Footprints:XIAO-nRF52840-SMD
Connections:
- net GND: now also U1.18 (GND), C43.1, D43.1 (VSS), D45.1 (VSS), D47.1 (VSS), D49.1 (VSS), D51.1 (VSS), D53.1 (VSS), D54.1 (VSS), D55.1 (VSS), D56.1 (VSS), D57.1 (VSS), D63.1 (VSS), D64.1 (VSS), D65.1 (VSS), D66.1 (VSS), D67.1 (VSS), D73.1 (VSS), D74.1 (VSS), D75.1 (VSS), D76.1 (VSS), D77.1 (VSS), D83.1 (VSS)
- net +3.3V: now reaches U1.12 (3V3_OUT)
- net +3.3V: now also C43.2, D43.3 (VDD), D45.3 (VDD), D47.3 (VDD), D49.3 (VDD), D51.3 (VDD), D53.3 (VDD), D54.3 (VDD), D55.3 (VDD), D56.3 (VDD), D57.3 (VDD), D63.3 (VDD), D64.3 (VDD), D65.3 (VDD), D66.3 (VDD), D67.3 (VDD), D73.3 (VDD), D74.3 (VDD), D75.3 (VDD), D76.3 (VDD), D77.3 (VDD), D83.3 (VDD)
- net LED DATA: now reaches U1.21 (NFC1)
- net LED DATA: now also R5.1
- new net: D63.4 (DOUT), D64.2 (DIN)
- new net: D64.4 (DOUT), D65.2 (DIN)
- new net: D55.4 (DOUT), D56.2 (DIN)
- new net: D56.4 (DOUT), D57.2 (DIN)
- new net: D49.4 (DOUT), D51.2 (DIN)
- new net: D51.4 (DOUT), D53.2 (DIN)
- new net: D53.4 (DOUT), D54.2 (DIN)
- new net: D54.4 (DOUT), D55.2 (DIN)
- new net: D73.4 (DOUT), D74.2 (DIN)
- new net: D74.4 (DOUT), D75.2 (DIN)
- new net: D57.4 (DOUT), D63.2 (DIN)
- new net: D75.4 (DOUT), D76.2 (DIN)
- new net: D76.4 (DOUT), D77.2 (DIN)
- new net: D43.4 (DOUT), D45.2 (DIN)
- new net: D45.4 (DOUT), D47.2 (DIN)
- new net: D43.2 (DIN), R5.2
- new net: D66.4 (DOUT), D67.2 (DIN)
- new net: D67.4 (DOUT), D73.2 (DIN)
- new net: D47.4 (DOUT), D49.2 (DIN)
- new net: D77.4 (DOUT), D83.2 (DIN)
- new net: D65.4 (DOUT), D66.2 (DIN)
- no-connect marks 8 -> 6
